File: pcb/HackPad - DuckyBoi  8K2R V1.kicad_sch (KiCad schematic)
At the start: 26 parts, among them SW1 RotaryEncoder_Switch, SW2 RotaryEncoder_Switch, SW3 SW_Push, SW4 SW_Push, SW5 SW_Push, SW6 SW_Push, SW7 SW_Push, SW8 SW_Push, SW9 SW_Push, U1 XIAO-RP2040-DIP

Commit message: update
Parts:
- U1: footprint ScottoKeebs_MCU:Seeed_XIAO_RP2040 -> OPL:XIAO-RP2040-DIP
Connections:
- net Col 0: now also U1.8 (GPIO1/RX); no longer U1.4 (GPIO29/ADC3/A3)
- net ROT1-A: now also U1.10 (GPIO4/MISO); no longer U1.2 (GPIO27/ADC1/A1)
- net ROT1-B: now also U1.11 (GPIO3/MOSI); no longer U1.3 (GPIO28/ADC2/A2)
- net ROT2-A: now also U1.2 (GPIO27/ADC1/A1); no longer U1.10 (GPIO4/MISO)
- net ROT2-B: now also U1.3 (GPIO28/ADC2/A2); no longer U1.11 (GPIO3/MOSI)
- net Row 1: now also U1.4 (GPIO29/ADC3/A3); no longer U1.8 (GPIO1/RX)
